File: kicad/cs_monitor/cs_monitor.kicad_pcb (KiCad board)
At the start: 2 copper layers, 60.9 x 44.9 mm, 130 parts, among them J1 Conn_01x01_Female, J2 Conn_01x01_Female, J3 Conn_01x01_Female, J4 Conn, J5 Conn_01x01_Female, J6 Conn_01x01_Female, J7 Conn_01x01_Female, J8 Conn_01x01_Female, J9 Conn_01x01_Female, Q1 5N10, Q2 Q_NMOS_GSD, T1 HY931147C, U1 W5500, U2 OPA354AIDBVR, U3 LM2733XMF, U4 LMR50410XDBVR, U5 NCP1117-3.3, U6 MCP1700x, Y1 25MHz, Y2 16

Commit message: удалено:       kicad/cs_monitor/#auto_saved_files# 	удалено:       kicad/cs_monitor/_autosave-cs_monitor.kicad_pcb 	удалено:       kicad/cs_monitor/_autosave-cs_monitor.kicad_sch 	удалено:       kicad/cs_monitor/cs_monitor-backups/cs_monitor-2025-07-08_182651.zip 	удалено:       kicad/cs_monitor/cs_monitor-backups/cs_monitor-2025-07-08_184111.zip 	удалено:       kicad/cs_monitor/cs_monitor-backups/cs_monitor-2025-07-18_140158.zip 	удалено:       kicad/cs_monitor/cs_monitor-backups/cs_monitor-2025-07-18_141545.zip 	изменено:      kicad/cs_monitor/cs_monitor.kicad_pcb 	изменено:      kicad/cs_monitor/cs_monitor.kicad_prl 	изменено:      kicad/cs_monitor/cs_monitor.kicad_sch 	удалено:       kicad/cs_monitor/~_autosave-cs_monitor.kicad_pcb.lck 	удалено:       kicad/cs_monitor/~cs_monitor.kicad_sch.lck 	изменено:      stm32cubeide/SC_Monitor/Core/Inc/networkint.h 	изменено:      stm32cubeide/SC_Monitor/Core/Src/network_int.c 	изменено:      stm32cubeide/SC_Monitor/Release/Core/Src/AD5245.d 	изменено:      stm32cubeide/SC_Monitor/Release/Core/Src/main.d 	изменено:      stm32cubeide/SC_Monitor/Release/Core/Src/network_int.cyclo 	изменено:      stm32cubeide/SC_Monitor/Release/Core/Src/network_int.d 	изменено:      stm32cubeide/SC_Monitor/Release/Core/Src/network_int.o 	изменено:      stm32cubeide/SC_Monitor/Release/Core/Src/network_int.su 	изменено:      stm32cubeide/SC_Monitor/Release/Core/Src/ssd1306.d 	изменено:      stm32cubeide/SC_Monitor/Release/Core/Src/stm32g4xx_hal_msp.d 	изменено:      stm32cubeide/SC_Monitor/Release/Core/Src/stm32g4xx_it.d 	изменено:      stm32cubeide/SC_Monitor/Release/Core/Src/subdir.mk 	изменено:      stm32cubeide/SC_Monitor/Release/SC_Monitor.elf 	изменено:      stm32cubeide/SC_Monitor/Release/SC_Monitor.list 	изменено:      stm32cubeide/SC_Monitor/Release/SC_Monitor.map 	изменено:      stm32cubeide/SC_Monitor/Release/objects.list 	изменено:      stm32cubeide/WEB_Interface/test_line.html  	stm32cubeide/SC_Monitor/Core/Inc/webpages.h  	stm32cu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
Parts:
- D8, R32: moved to F.Cu
- moved D8 47.1 mm to (134.3, 65.5), turned to -90 degrees
- moved R32 45.0 mm to (132.8, 65.5)
Routing:
- net +5V: track 108.3 -> 109.7 mm
- net MISO: track 7.24 -> 7.81 mm

Commit message: удалено:       kicad/cs_monitor/cs_monitor-backups/cs_monitor-2025-07-08_184829.zip 	удалено:       kicad/cs_monitor/cs_monitor-backups/cs_monitor-2025-07-08_185838.zip 	изменено:      kicad/cs_monitor/cs_monitor.kicad_pcb 	изменено:      kicad/cs_monitor/cs_monitor.kicad_pro 	изменено:      kicad/cs_monitor/cs_monitor.kicad_sch 	изменено:      kicad/cs_monitor/gerber/cs_monitor.drl 	удалено:       kicad/cs_monitor/gerber/cs_monitor_T01_0.30mm.gcode 	удалено:       kicad/cs_monitor/gerber/cs_monitor_T02_0.40mm.gcode 	удалено:       kicad/cs_monitor/gerber/cs_monitor_T03_0.70mm.gcode 	удалено:       kicad/cs_monitor/gerber/cs_monitor_T04_0.76mm.gcode 	удалено:       kicad/cs_monitor/gerber/cs_monitor_T05_1.00mm.gcode 	удалено:       kicad/cs_monitor/gerber/cs_monitor_T06_1.63mm.gcode 	изменено:      stm32cubeide/SC_Monitor/.mxproject 	изменено:      stm32cubeide/SC_Monitor/.settings/language.settings.xml 	изменено:      stm32cubeide/SC_Monitor/Core/Inc/main.h 	изменено:      stm32cubeide/SC_Monitor/Core/Src/main.c 	изменено:      stm32cubeide/SC_Monitor/Release/Core/Src/main.cyclo 	изменено:      stm32cubeide/SC_Monitor/Release/Core/Src/main.o 	изменено:      stm32cubeide/SC_Monitor/Release/Core/Src/main.su 	изменено:      stm32cubeide/SC_Monitor/Release/SC_Monitor.elf 	изменено:      stm32cubeide/SC_Monitor/Release/SC_Monitor.list 	изменено:      stm32cubeide/SC_Monitor/Release/SC_Monitor.map 	изменено:      stm32cubeide/SC_Monitor/SC_Monitor Release.launch 	изменено:      stm32cubeide/SC_Monitor/SC_Monitor.ioc
Parts:
- added C52: 10u, Capacitor_SMD:C_0402_1005Metric, B.Cu at (109.9, 48.8)
- C24: moved to F.Cu
- R24: moved to B.Cu
- moved C35 19.4 mm to (124.5, 65.0), turned to -90 degrees
- moved J8 15.1 mm to (124.5, 66.5)
- moved C29 15.1 mm to (120.7, 65.0), turned to -90 degrees
- moved R29 14.9 mm to (122.6, 65.8), turned to 90 degrees
- moved C50 11.5 mm to (130.9, 51.2), turned to 0 degrees
- moved D3 9.06 mm to (117.5, 70.1), turned to 180 degrees
- moved L5 8.95 mm to (120.8, 69.0), turned to 90 degrees
- moved R39 8.92 mm to (121.6, 65.0), turned to 180 degrees
- moved U6 8.30 mm to (131.1, 53.9), turned to 0 degrees
- moved D8 8.03 mm to (128.1, 60.4), turned to 0 degrees
- moved C27 7.24 mm to (117.1, 67.5), turned to 0 degrees
- moved C26 6.96 mm to (116.3, 64.1), turned to 0 degrees
- moved C49 6.31 mm to (128.1, 53.9), turned to -90 degrees
- moved Q2 6.19 mm to (121.6, 67.8), turned to -90 degrees
- moved R18 6.13 mm to (116.3, 65.6), turned to 180 degrees
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Connections:
- D2 pad 25: INT_ETH -> SS_ETH
- D2 pad 26: SS_ETH -> INT_ETH
Routing:
- net GND: track 152.1 -> 141.6 mm, vias 11 -> 14
- net +5V: track 109.7 -> 116.4 mm
- net Sound: track 17.7 -> 11.1 mm
- net Net-(BZ1-+): track 2.48 -> 8.02 mm
- net SCL: track 34.3 -> 30.0 mm
- net +3V3: track 141.3 -> 144.3 mm
- net Net-(D2-pa6): track 10.2 -> 7.41 mm
- net Pulse: track 22.6 -> 19.9 mm
- net AdjHV: track 18.5 -> 16.0 mm, vias 2 -> 1
- net Analog: track 14.5 -> 12.2 mm
- net SDA: track 39.5 -> 37.6 mm
- net Net-(U3-FB): track 5.84 -> 4.53 mm, vias 0 -> 1
- net +30v: track 3.64 -> 2.53 mm
- net -PoE: track 12.9 -> 12.0 mm
- net Net-(D3-K): track 7.73 -> 8.57 mm
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Other:
- board size 60.9 x 44.9 mm -> 57.5 x 44.9 mm

Commit message: новый файл:    kicad/cs_monitor/bom/ibom.html 	изменено:      kicad/cs_monitor/cs_monitor.kicad_pcb 	изменено:      kicad/cs_monitor/cs_monitor.kicad_sch 	изменено:      stm32cubeide/SC_Monitor/.mxproject 	изменено:      stm32cubeide/SC_Monitor/.settings/language.settings.xml 	изменено:      stm32cubeide/SC_Monitor/Core/Src/main.c 	изменено:      stm32cubeide/SC_Monitor/Release/Core/Src/main.cyclo 	изменено:      stm32cubeide/SC_Monitor/Release/Core/Src/main.o 	изменено:      stm32cubeide/SC_Monitor/Release/Core/Src/main.su 	изменено:      stm32cubeide/SC_Monitor/Release/SC_Monitor.elf 	изменено:      stm32cubeide/SC_Monitor/Release/SC_Monitor.list 	изменено:      stm32cubeide/SC_Monitor/Release/SC_Monitor.map 	изменено:      stm32cubeide/SC_Monitor/SC_Monitor.ioc
Parts:
- C26: value 220p -> 82p
- R18: value 117k -> 120k
- R19: value 5.1k -> 4.3k
- R24: value 50k -> 33k
- R26: value 1.02k -> 1k
Changed lines of the file:
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@@
 			)
 		)
-		(property "Value" "5.1k"
+		(property "Value" "4.3k"
 			(at 0 1.43 0)
 			(layer "F.Fab")
@@
 			)
 		)
-		(property "Value" "117k"
+		(property "Value" "120k"
 			(at 0 1.43 0)
 			(layer "F.Fab")
@@
 			)
 		)
-		(property "Value" "220p"
+		(property "Value" "82p"
 			(at 0 1.43 0)
 			(layer "F.Fab")
@@
 			)
 		)
-		(property "Value" "50k"
+		(property "Value" "33k"
 			(at 0 -1.43 90)
 			(layer "B.Fab")
@@
 			)
 		)
-		(property "Value" "1.02k"
+		(property "Value" "1k"
 			(at 0 -1.43 90)
 			(layer "B.Fab")

Commit message: удалено:       kicad/cs_monitor/cs_monitor-backups/cs_monitor-2025-07-09_181433.zip 	удалено:       kicad/cs_monitor/cs_monitor-backups/cs_monitor-2025-07-09_181946.zip 	изменено:      kicad/cs_monitor/cs_monitor.kicad_pcb 	изменено:      kicad/cs_monitor/cs_monitor.kicad_prl 	изменено:      stm32cubeide/SC_Monitor/Core/Inc/webpages.h 	изменено:      stm32cubeide/SC_Monitor/Core/Src/network_int.c 	изменено:      stm32cubeide/SC_Monitor/Release/Core/Src/network_int.o 	изменено:      stm32cubeide/SC_Monitor/Release/SC_Monitor.elf 	изменено:      stm32cubeide/SC_Monitor/Release/SC_Monitor.list 	изменено:      stm32cubeide/SC_Monitor/Release/SC_Monitor.map
Parts:
- moved R37 0.24 mm to (116.2, 45.3)
Changed lines of the file:
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@@
 	(footprint "Resistor_SMD:R_0402_1005Metric"
 		(layer "F.Cu")
-		(at 116.24 45.56)
+		(at 116.24 45.32)
 		(descr "Resistor SMD 0402 (1005 Metric), square (rectangular) end terminal, IPC-7351 nominal, (Body size source: IPC-SM-782 page 72, https://www.pcb-3d.com/wordpress/wp-content/uploads/ipc-sm-782a_amendment_1_and_2.pdf), generated with kicad-footprint-generator")
 		(tags "resistor")
@@
 	)
 	(segment
-		(start 118.322842 44.687158)
-		(end 118.167157 44.842843)
-		(width 0.2)
-		(layer "F.Cu")
-		(net 8)
-	)
-	(segment
 		(start 80.94625 54.59625)
 		(end 82.829607 52.712893)
@@
 	)
 	(segment
-		(start 89.58 81.02)
-		(end 89.71 81.15)
+		(start 116.515736 45.085736)
+		(end 116.75 45.32)
 		(width 0.2)
 		(layer "F.Cu")
@@
 	)
 	(segment
-		(start 116.34 44.96)
-		(end 116.34 45.15)
+		(start 89.58 81.02)
+		(end 89.71 81.15)
 		(width 0.2)
 		(layer "F.Cu")
@@
 	)
 	(segment
+		(start 118.155736 45.144264)
+		(end 118.264264 45.035736)
+		(width 0.2)
+		(layer "F.Cu")
+		(net 8)
+	)
+	(segment
 		(start 118.97 59.2)
 		(end 118.97 59.39825)
@@
 	)
 	(segment
+		(start 116.34 43.53)
+		(end 116.34 44.661472)
+		(width 0.2)
+		(layer "F.Cu")
+		(net 8)
+	)
+	(segment
 		(start 92.322893 52.712893)
 		(end 93.007107 53.397107)
@@
 	)
 	(segment
-		(start 116.34 45.15)
-		(end 116.75 45.56)
-		(width 0.2)
-		(layer "F.Cu")
-		(net 8)
-	)
-	(segment
 		(start 112.677107 54.327107)
 		(end 112.152893 53.802893)
@@
 	)
 	(segment
-		(start 116.34 43.53)
-		(end 116.34 44.96)
+		(start 116.83 45.4)
+		(end 116.75 45.32)
 		(width 0.2)
 		(layer "F.Cu")
@@
 	)
 	(segment
+		(start 116.75 45.32)
+		(end 117.731472 45.32)
+		(width 0.2)
+		(layer "F.Cu")
+		(net 8)
+	)
+	(segment
 		(start 93.714214 53.69)
 		(end 101.21 53.69)
@@
 	)
 	(segment
-		(start 83.536714 52.42)
-		(end 91.615786 52.42)
+		(start 118.44 44.611472)
+		(end 118.44 43.53)
 		(width 0.2)
 		(layer "F.Cu")
@@
 	)
 	(segment
-		(start 117.884315 44.96)
-		(end 116.34 44.96)
+		(start 83.536714 52.42)
+		(end 91.615786 52.42)
 		(width 0.2)
 		(layer "F.Cu")
@@
 	)
 	(segment
-		(start 118.44 43.53)
-		(end 118.44 44.404315)
-		(width 0.2)
-		(layer "F.Cu")
-		(net 8)
-	)
-	(segment
 		(start 116.44 57.65325)
 		(end 117.091879 57.65325)
@@
 	)
 	(via
-		(at 116.63 45.25)
+		(at 117.45 45.4)
 		(size 0.8)
 		(drill 0.4)
@@
 	)
 	(arc
+		(start 118.155736 45.144264)
+		(mid 117.961082 45.274328)
+		(end 117.731472 45.32)
+		(width 0.2)
+		(layer "F.Cu")
+		(net 8)
+	)
+	(arc
+		(start 118.44 44.611472)
+		(mid 118.394328 44.841082)
+		(end 118.264264 45.035736)
+		(width 0.2)
+		(layer "F.Cu")
+		(net 8)
+	)
+	(arc
 		(start 112.677107 54.327107)
 		(mid 112.89388 54.65153)
@@
 	)
 	(arc
-		(start 118.167157 44.842843)
-		(mid 118.037388 44.929552)
-		(end 117.884315 44.96)
+		(start 116.34 44.661472)
+		(mid 116.385672 44.891082)
+		(end 116.515736 45.085736)
 		(width 0.2)
 		(layer "F.Cu")
@@
 	)
 	(arc
-		(start 118.44 44.404315)
-		(mid 118.409552 44.557389)
-		(end 118.322842 44.687158)
-		(width 0.2)
-		(layer "F.Cu")
-		(net 8)
-	)
-	(arc
 		(start 111.86 53.095786)
 		(mid 111.93612 53.478469)
@@
 	)
 	(segment
+		(start 117.870393 55.899607)
+		(end 117.937107 55.832893)
+		(width 0.2)
+		(layer "B.Cu")
+		(net 8)
+	)
+	(segment
+		(start 116.83 56.1925)
+		(end 117.163286 56.1925)
+		(width 0.2)
+		(layer "B.Cu")
+		(net 8)
+	)
+	(segment
 		(start 102.74625 54.16)
 		(end 102.74625 55.00625)
@@
 	)
 	(segment
-		(start 116.63 45.25)
-		(end 116.63 47.055786)
+		(start 80.94625 43.88625)
+		(end 79.842893 44.989607)
 		(width 0.2)
 		(layer "B.Cu")
@@
 	)
 	(segment
-		(start 80.94625 43.88625)
-		(end 79.842893 44.989607)
+		(start 116.69 47.281472)
+		(end 116.69 47.138528)
 		(width 0.2)
 		(layer "B.Cu")
@@
 	)
 	(segment
-		(start 117.163286 56.1925)
-		(end 116.83 56.1925)
-		(width 0.2)
-		(layer "B.Cu")
-		(net 8)
-	)
-	(segment
 		(start 110.145893 57.049143)
 		(end 110.457107 57.360357)
@@
 	)
 	(segment
-		(start 118.23 49.484214)
-		(end 118.23 55.125786)
+		(start 117.937107 48.777107)
+		(end 116.865736 47.705736)
 		(width 0.2)
 		(layer "B.Cu")
@@
 	)
 	(segment
-		(start 116.922893 47.762893)
-		(end 117.937107 48.777107)
-		(width 0.2)
-		(layer "B.Cu")
-		(net 8)
-	)
-	(segment
 		(start 102.74625 53.617964)
 		(end 102.74625 54.16)
@@
 	)
 	(segment
-		(start 117.937107 55.832893)
-		(end 117.870393 55.899607)
+		(start 117.45 45.881472)
+		(end 117.45 45.4)
+		(width 0.2)
+		(layer "B.Cu")
+		(net 8)
+	)
+	(segment
+		(start 116.865736 46.714264)
+		(end 117.274264 46.305736)
 		(width 0.2)
 		(layer "B.Cu")
@@
 	)
 	(segment
+		(start 118.23 55.125786)
+		(end 118.23 49.484214)
+		(width 0.2)
+		(layer "B.Cu")
+		(net 8)
+	)
+	(segment
 		(start 106.34 49.61)
 		(end 103.039143 52.910857)
@@
 	)
 	(arc
+		(start 118.23 49.484214)
+		(mid 118.15388 49.101531)
+		(end 117.937107 48.777107)
+		(width 0.2)
+		(layer "B.Cu")
+		(net 8)
+	)
+	(arc
 		(start 108.741986 49.418014)
 		(mid 108.547332 49.548078)
@@
 	)
 	(arc
-		(start 103.039143 52.910857)
-		(mid 102.82237 53.23528)
-		(end 102.74625 53.617964)
-		(width 0.6)
+		(start 117.937107 55.832893)
+		(mid 118.15388 55.50847)
+		(end 118.23 55.125786)
+		(width 0.2)
 		(layer "B.Cu")
 		(net 8)
 	)
 	(arc
-		(start 116.63 47.055786)
-		(mid 116.70612 47.438469)
-		(end 116.922893 47.762893)
-		(width 0.2)
+		(start 103.039143 52.910857)
+		(mid 102.82237 53.23528)
+		(end 102.74625 53.617964)
+		(width 0.6)
 		(layer "B.Cu")
 		(net 8)
 	)
 	(arc
-		(start 117.937107 48.777107)
-		(mid 118.15388 49.101531)
-		(end 118.23 49.484214)
+		(start 117.45 45.881472)
+		(mid 117.404328 46.111082)
+		(end 117.274264 46.305736)
 		(width 0.2)
 		(layer "B.Cu")
@@
 	)
 	(arc
-		(start 117.937107 55.832893)
-		(mid 118.15388 55.50847)
-		(end 118.23 55.125786)
+		(start 116.69 47.138528)
+		(mid 116.735672 46.908918)
+		(end 116.865736 46.714264)
 		(width 0.2)
 		(layer "B.Cu")
@@
 	)
 	(arc
+		(start 116.69 47.281472)
+		(mid 116.735672 47.511082)
+		(end 116.865736 47.705736)
+		(width 0.2)
+		(layer "B.Cu")
+		(net 8)
+	)
+	(arc
 		(start 110.145893 57.049143)
 		(mid 109.82147 56.83237)
@@
 	)
 	(segment
-		(start 115.64 43.53)
-		(end 115.64 45.47)
+		(start 115.64 45.23)
+		(end 115.73 45.32)
 		(width 0.2)
 		(layer "F.Cu")
@@
 	)
 	(segment
-		(start 115.64 45.47)
-		(end 115.73 45.56)
+		(start 115.64 43.53)
+		(end 115.64 45.23)
 		(width 0.2)
 		(layer "F.Cu")
@@
 		(polygon
 			(pts
-				(xy 119.24 40.17) (xy 119.24 64.460155) (xy 135.713795 64.477147) (xy 135.693836 63.808502) (xy 119.99 63.8)
-				(xy 120.08 63.89) (xy 120.07 40.17) (xy 119.25 40.17)
+				(xy 119.24 46.89) (xy 119.24 64.460155) (xy 135.713795 64.477147) (xy 135.693836 63.808502) (xy 119.99 63.8)
+				(xy 120.08 63.89) (xy 120.072833 46.89)
 			)
 		)
@@
 		(polygon
 			(pts
-				(xy 115.07 48.21) (xy 116.75 48.21) (xy 116.75 48.02) (xy 114.86 48.02) (xy 114.86 53.284334) (xy 115.09 53.66)
+				(xy 115.042941 40.836471) (xy 114.86 40.670953) (xy 114.86 53.284334) (xy 115.09 53.66)
 			)
 		)

Commit message: удалено:       kicad/cs_monitor/cs_monitor-backups/cs_monitor-2025-07-09_183647.zip 	удалено:       kicad/cs_monitor/cs_monitor-backups/cs_monitor-2025-07-09_190248.zip 	изменено:      kicad/cs_monitor/cs_monitor.kicad_pcb 	изменено:      kicad/cs_monitor/cs_monitor.kicad_sch
Parts:
- R18: value 120k -> 330k
- R19: value 4.3k -> 13k
- R29: value 20k -> 1k
Changed lines of the file:
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@@
 			)
 		)
-		(property "Value" "4.3k"
+		(property "Value" "13k"
 			(at 0 1.43 0)
 			(layer "F.Fab")
@@
 			)
 		)
-		(property "Value" "120k"
+		(property "Value" "330k"
 			(at 0 1.43 0)
 			(layer "F.Fab")
@@
 			)
 		)
-		(property "Value" "20k"
+		(property "Value" "1k"
 			(at 0 1.43 90)
 			(layer "F.Fab")

Commit message: удалено:       kicad/cs_monitor/cs_monitor-backups/cs_monitor-2025-07-09_190842.zip 	удалено:       kicad/cs_monitor/cs_monitor-backups/cs_monitor-2025-07-11_220437.zip 	удалено:       kicad/cs_monitor/cs_monitor-backups/cs_monitor-2025-07-11_223758.zip 	удалено:       kicad/cs_monitor/cs_monitor-backups/cs_monitor-2025-07-11_224909.zip 	изменено:      kicad/cs_monitor/cs_monitor.kicad_pcb 	изменено:      kicad/cs_monitor/cs_monitor.kicad_prl 	изменено:      stm32cubeide/SC_Monitor/.mxproject 	изменено:      stm32cubeide/SC_Monitor/Core/Inc/stm32g4xx_hal_conf.h 	изменено:      stm32cubeide/SC_Monitor/Core/Inc/stm32g4xx_it.h 	изменено:      stm32cubeide/SC_Monitor/Core/Src/main.c 	изменено:      stm32cubeide/SC_Monitor/Core/Src/stm32g4xx_hal_msp.c 	изменено:      stm32cubeide/SC_Monitor/Core/Src/stm32g4xx_it.c 	изменено:      stm32cubeide/SC_Monitor/Release/Core/Src/AD5245.d 	изменено:      stm32cubeide/SC_Monitor/Release/Core/Src/main.cyclo 	изменено:      stm32cubeide/SC_Monitor/Release/Core/Src/main.d 	изменено:      stm32cubeide/SC_Monitor/Release/Core/Src/main.o 	изменено:      stm32cubeide/SC_Monitor/Release/Core/Src/main.su 	изменено:      stm32cubeide/SC_Monitor/Release/Core/Src/network_int.d 	изменено:      stm32cubeide/SC_Monitor/Release/Core/Src/ssd1306.d 	изменено:      stm32cubeide/SC_Monitor/Release/Core/Src/stm32g4xx_hal_msp.cyclo 	изменено:      stm32cubeide/SC_Monitor/Release/Core/Src/stm32g4xx_hal_msp.d 	изменено:      stm32cubeide/SC_Monitor/Release/Core/Src/stm32g4xx_hal_msp.o 	изменено:      stm32cubeide/SC_Monitor/Release/Core/Src/stm32g4xx_hal_msp.su 	изменено:      stm32cubeide/SC_Monitor/Release/Core/Src/stm32g4xx_it.cyclo 	изменено:      stm32cubeide/SC_Monitor/Release/Core/Src/stm32g4xx_it.d 	изменено:      stm32cubeide/SC_Monitor/Release/Core/Src/stm32g4xx_it.o 	изменено:      stm32cubeide/SC_Monitor/Release/Core/Src/stm32g4xx_it.su 	изменено:      stm32cubeide/SC_Monitor/Release/Core/Src/system_stm32g4xx.d 	изменено:      stm32cubeide/SC_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
Parts:
- moved R24 3.00 mm to (117.7, 64.9), turned to 0 degrees
- moved R29 2.30 mm to (123.1, 68.0), turned to 0 degrees
- moved C14 1.66 mm to (100.5, 45.0), turned to 0 degrees
- moved R3 1.59 mm to (121.8, 55.2)
- moved C26 1.33 mm to (117.6, 64.2)
- moved R18 1.33 mm to (117.6, 65.7)
- moved C35 1.27 mm to (123.2, 65.0)
- moved R19 1.25 mm to (114.7, 65.0)
- moved J8 0.78 mm to (123.7, 66.5)
- moved Q2 0.67 mm to (121.0, 68.2)
- moved R39 0.67 mm to (121.0, 65.4)
- moved D6 0.48 mm to (101.6, 66.6)
- moved L1 0.41 mm to (100.7, 52.8)
- moved C10 0.35 mm to (105.6, 44.6)
- moved C12 0.34 mm to (104.5, 44.5)
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Routing:
- net GND: track 141.6 -> 153.8 mm
- net INT_ETH: track 12.6 -> 9.99 mm
- net /3.3VA: track 28.0 -> 30.5 mm
- net MOSI: track 7.64 -> 5.53 mm
- net Net-(D2-pa6): track 7.41 -> 9.20 mm
- net +5V: track 116.4 -> 114.7 mm
- net MISO: track 7.76 -> 6.11 mm
- net +3V3: track 144.2 -> 145.2 mm
- net Adj: track 5.49 -> 4.45 mm
- net Net-(U1-RXP): track 10.4 -> 11.4 mm
- net +30v: track 2.53 -> 1.71 mm
- net Net-(D6-A): track 3.77 -> 3.01 mm
- net AdjHV: track 16.0 -> 15.3 mm
- net SCLK: track 7.20 -> 6.48 mm
- net SCL: track 30.0 -> 30.6 mm
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
Commit message: изменено:      kicad/cs_monitor/cs_monitor.kicad_pcb 	изменено:      kicad/cs_monitor/cs_monitor.kicad_sch 	изменено:      stm32cubeide/SC_Monitor/Core/Inc/main.h 	изменено:      stm32cubeide/SC_Monitor/Core/Src/main.c 	изменено:      stm32cubeide/SC_Monitor/Release/Core/Src/main.o 	изменено:      stm32cubeide/SC_Monitor/Release/SC_Monitor.elf 	изменено:      stm32cubeide/SC_Monitor/Release/SC_Monitor.list 	изменено:      stm32cubeide/SC_Monitor/Release/SC_Monitor.map 	изменено:      stm32cubeide/SC_Monitor/SC_Monitor.ioc
Parts:
- R12: value 3k -> 3k*
Changed lines of the file:
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@@
 			)
 		)
-		(property "Value" "3k"
+		(property "Value" "3k*"
 			(at 0 -1.43 0)
 			(layer "B.Fab")
